File: blestack01/blestack01.kicad_sch (KiCad schematic)
At the start: 17 parts, among them J1 IO, P1 USB_C_Plug_USB2.0, SW1 USER, SW2 RST, U1 AP2112K-3.3, U2 ESP32-C3-MINI-1

Commit message: Gamepad Stack
Parts:
- added R?: 10k, Resistor_SMD:R_0402_1005Metric, symbol Device:R
Connections:
- net VBUS: now also R?.2
- net at U1.3 (EN): now also R?.1
- no-connect marks 3 -> 2
Changed lines of the file:
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@@
   (junction (at 180.848 114.3) (diameter 0) (color 0 0 0 0)
+  )
+  (junction (at 53.086 24.384) (diameter 0) (color 0 0 0 0)
   )
   (junction (at 82.55 24.384) (diameter 0) (color 0 0 0 0)
@@
   (no_connect (at 42.672 29.464))
   (no_connect (at 42.672 32.004))
-  (no_connect (at 61.976 26.924))
   (wire (pts (xy 219.456 66.04) (xy 219.456 67.056))
     (stroke (width 0) (type default) (color 0 0 0 0))
@@
     (stroke (width 0) (type default) (color 0 0 0 0))
   )
-  (wire (pts (xy 47.244 24.384) (xy 61.976 24.384))
+  (wire (pts (xy 47.244 24.384) (xy 53.086 24.384))
     (stroke (width 0) (type default) (color 0 0 0 0))
   )
@@
     (stroke (width 0) (type default) (color 0 0 0 0))
   )
+  (wire (pts (xy 53.086 24.384) (xy 53.086 26.924))
+    (stroke (width 0) (type default) (color 0 0 0 0))
+  )
   (wire (pts (xy 205.74 114.046) (xy 205.74 116.586))
     (stroke (width 0) (type default) (color 0 0 0 0))
@@
     (stroke (width 0) (type default) (color 0 0 0 0))
   )
+  (wire (pts (xy 61.214 26.924) (xy 61.976 26.924))
+    (stroke (width 0) (type default) (color 0 0 0 0))
+  )
   (wire (pts (xy 122.428 113.03) (xy 124.46 113.03))
     (stroke (width 0) (type default) (color 0 0 0 0))
@@
     (stroke (width 0) (type default) (color 0 0 0 0))
   )
+  (wire (pts (xy 53.086 24.384) (xy 61.976 24.384))
+    (stroke (width 0) (type default) (color 0 0 0 0))
+  )
   (wire (pts (xy 69.596 34.544) (xy 69.596 35.56))
     (stroke (width 0) (type default) (color 0 0 0 0))
@@
   )
   (wire (pts (xy 179.07 114.3) (xy 180.848 114.3))
+    (stroke (width 0) (type default) (color 0 0 0 0))
+  )
+  (wire (pts (xy 53.594 26.924) (xy 53.086 26.924))
     (stroke (width 0) (type default) (color 0 0 0 0))
   )
@@
     (pin "1")
   )
+  (symbol (lib_id "Device:R") (at 57.404 26.924 270) (unit 1)
+    (in_bom yes) (on_board yes)
+    (property "Reference" "R?" (id 0) (at 57.404 29.21 90))
+    (property "Value" "10k" (id 1) (at 57.404 31.242 90))
+    (property "Footprint" "Resistor_SMD:R_0402_1005Metric" (id 2) (at 57.404 25.146 90)
+      (effects (font (size 1.27 1.27)) hide)
+    )
+    (property "Datasheet" "" (id 3) (at 57.404 26.924 0)
+      (effects (font (size 1.27 1.27)) hide)
+    )
+    (property "LCSC" "C25744" (id 4) (at 57.404 26.924 90)
+      (effects (font (size 1.27 1.27)) hide)
+    )
+    (pin "1")
+    (pin "2")
+  )
   (symbol (lib_id "Device:R") (at 114.046 59.436 0) (unit 1)
     (in_bom yes) (on_board yes) (fields_autoplaced)
@@
       (reference "R5") (unit 1) (value "1k") (footprint "Resistor_SMD:R_0402_1005Metric")
     )
+    (path "/5ff8f998-a8ba-4b02-b757-369a40737a4b"
+      (reference "R?") (unit 1) (value "10k") (footprint "Resistor_SMD:R_0402_1005Metric")
+    )
     (path "/5b56d039-6401-46e7-bb94-fe3df74cfb71"
